File: hardware/PicoDAC/PicoDAC.kicad_sch (KiCad schematic)
At the start: 45 parts, among them CN1 PJ-327A 5JJ, U1 CS43131-CNZR, U2 XIAO-RP2350-DIP, U3 PCA9306DCUR, U4 SN74AXC4T245PWR, U5 XTPS7A2018, U7 74AHCT1G125GV

Commit message: optimized parts (this reduced cost a lot)
Parts:
- C1, C15, C16, C2, C3: LCSC Part C60474 -> C1525; MPN CC0402KRX7R7BB104 -> CL05B104KO5NNNC; Manufacturer (none) -> Samsung Electro-Mechanics
- R1, R2, R3: LCSC Part C60490 -> C25744; MPN RC0402FR-0710KL -> 0402WGF1002TCE; Manufacturer (none) -> UNI-ROYAL(Uniroyal Elec)
- R5, R6, R7, R8: LCSC Part C105871 -> C25900; MPN RC0402FR-074K7L -> 0402WGF4701TCE; Manufacturer (none) -> UNI-ROYAL(Uniroyal Elec)
- R9: LCSC Part C105875 -> C25104; MPN RC0402FR-07330RL -> 0402WGF3300TCE; Manufacturer (none) -> UNI-ROYAL(Uniroyal Elec)
Changed lines of the file:
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@@
 			)
 		)
-		(property "Datasheet" "https://www.lcsc.com/datasheet/C60474.pdf"
+		(property "Datasheet" "https://jlcpcb.com/api/file/downloadByFileSystemAccessId/8579707269996871680"
 			(at 38.1 124.46 0)
 			(effects
@@
 			)
 		)
-		(property "LCSC Part" "C60474"
+		(property "LCSC Part" "C1525"
 			(at 38.1 124.46 0)
 			(effects
@@
 			)
 		)
-		(property "MPN" "CC0402KRX7R7BB104"
+		(property "MPN" "CL05B104KO5NNNC"
+			(at 38.1 124.46 0)
+			(effects
+				(font
+					(size 1.27 1.27)
+				)
+				(hide yes)
+			)
+		)
+		(property "Manufacturer" "Samsung Electro-Mechanics"
 			(at 38.1 124.46 0)
 			(effects
@@
 			)
 		)
-		(property "Datasheet" "https://www.lcsc.com/datasheet/C105871.pdf"
+		(property "Datasheet" "https://jlcpcb.com/api/file/downloadByFileSystemAccessId/8579705941367193600"
 			(at 139.7 196.85 0)
 			(effects
@@
 			)
 		)
-		(property "LCSC Part" "C105871"
+		(property "LCSC Part" "C25900"
+			(at 139.7 196.85 90)
+			(effects
+				(font
+					(size 1.27 1.27)
+				)
+				(hide yes)
+			)
+		)
+		(property "MPN" "0402WGF4701TCE"
 			(at 139.7 196.85 90)
 			(effects
@@
 			)
 		)
-		(property "MPN" "RC0402FR-074K7L"
+		(property "Manufacturer" "UNI-ROYAL(Uniroyal Elec)"
 			(at 139.7 196.85 90)
 			(effects
@@
 			)
 		)
-		(property "Datasheet" "https://www.lcsc.com/datasheet/C60490.pdf"
+		(property "Datasheet" "https://jlcpcb.com/api/file/downloadByFileSystemAccessId/8556212101498380288"
 			(at 41.91 182.88 0)
 			(effects
@@
 			)
 		)
-		(property "LCSC Part" "C60490"
+		(property "LCSC Part" "C25744"
 			(at 41.91 182.88 0)
 			(effects
@@
 			)
 		)
-		(property "MPN" "RC0402FR-0710KL"
+		(property "MPN" "0402WGF1002TCE"
+			(at 41.91 182.88 0)
+			(effects
+				(font
+					(size 1.27 1.27)
+				)
+				(hide yes)
+			)
+		)
+		(property "Manufacturer" "UNI-ROYAL(Uniroyal Elec)"
 			(at 41.91 182.88 0)
 			(effects
@@
 			)
 		)
-		(property "Datasheet" "https://www.lcsc.com/datasheet/C60474.pdf"
+		(property "Datasheet" "https://jlcpcb.com/api/file/downloadByFileSystemAccessId/8579707269996871680"
 			(at 107.95 196.85 0)
 			(effects
@@
 			)
 		)
-		(property "LCSC Part" "C60474"
+		(property "LCSC Part" "C1525"
+			(at 107.95 196.85 0)
+			(effects
+				(font
+					(size 1.27 1.27)
+				)
+				(hide yes)
+			)
+		)
+		(property "MPN" "CL05B104KO5NNNC"
 			(at 107.95 196.85 0)
 			(effects
@@
 			)
 		)
-		(property "MPN" "CC0402KRX7R7BB104"
+		(property "Manufacturer" "Samsung Electro-Mechanics"
 			(at 107.95 196.85 0)
 			(effects
@@
 			)
 		)
-		(property "Datasheet" "https://www.lcsc.com/datasheet/C60490.pdf"
+		(property "Datasheet" "https://jlcpcb.com/api/file/downloadByFileSystemAccessId/8556212101498380288"
 			(at 163.83 100.33 0)
 			(effects
@@
 			)
 		)
-		(property "LCSC Part" "C60490"
+		(property "LCSC Part" "C25744"
+			(at 163.83 100.33 0)
+			(effects
+				(font
+					(size 1.27 1.27)
+				)
+				(hide yes)
+			)
+		)
+		(property "MPN" "0402WGF1002TCE"
 			(at 163.83 100.33 0)
 			(effects
@@
 			)
 		)
-		(property "MPN" "RC0402FR-0710KL"
+		(property "Manufacturer" "UNI-ROYAL(Uniroyal Elec)"
 			(at 163.83 100.33 0)
 			(effects
@@
 			)
 		)
-		(property "Datasheet" "https://www.lcsc.com/datasheet/C60474.pdf"
+		(property "Datasheet" "https://jlcpcb.com/api/file/downloadByFileSystemAccessId/8579707269996871680"
 			(at 33.02 124.46 0)
 			(effects
@@
 			)
 		)
-		(property "LCSC Part" "C60474"
+		(property "LCSC Part" "C1525"
 			(at 33.02 124.46 0)
 			(effects
@@
 			)
 		)
-		(property "MPN" "CC0402KRX7R7BB104"
+		(property "MPN" "CL05B104KO5NNNC"
+			(at 33.02 124.46 0)
+			(effects
+				(font
+					(size 1.27 1.27)
+				)
+				(hide yes)
+			)
+		)
+		(property "Manufacturer" "Samsung Electro-Mechanics"
 			(at 33.02 124.46 0)
 			(effects
@@
 			)
 		)
-		(property "Datasheet" "https://www.lcsc.com/datasheet/C105871.pdf"
+		(property "Datasheet" "https://jlcpcb.com/api/file/downloadByFileSystemAccessId/8579705941367193600"
 			(at 209.55 196.85 0)
 			(effects
@@
 			)
 		)
-		(property "LCSC Part" "C105871"
+		(property "LCSC Part" "C25900"
+			(at 209.55 196.85 90)
+			(effects
+				(font
+					(size 1.27 1.27)
+				)
+				(hide yes)
+			)
+		)
+		(property "MPN" "0402WGF4701TCE"
 			(at 209.55 196.85 90)
 			(effects
@@
 			)
 		)
-		(property "MPN" "RC0402FR-074K7L"
+		(property "Manufacturer" "UNI-ROYAL(Uniroyal Elec)"
 			(at 209.55 196.85 90)
 			(effects
@@
 			)
 		)
-		(property "Datasheet" "https://www.lcsc.com/datasheet/C60474.pdf"
+		(property "Datasheet" "https://jlcpcb.com/api/file/downloadByFileSystemAccessId/8579707269996871680"
 			(at 34.29 196.85 0)
 			(effects
@@
 			)
 		)
-		(property "LCSC Part" "C60474"
+		(property "LCSC Part" "C1525"
 			(at 34.29 196.85 0)
 			(effects
@@
 			)
 		)
-		(property "MPN" "CC0402KRX7R7BB104"
+		(property "MPN" "CL05B104KO5NNNC"
+			(at 34.29 196.85 0)
+			(effects
+				(font
+					(size 1.27 1.27)
+				)
+				(hide yes)
+			)
+		)
+		(property "Manufacturer" "Samsung Electro-Mechanics"
 			(at 34.29 196.85 0)
 			(effects
@@
 			)
 		)
-		(property "Datasheet" "https://www.lcsc.com/datasheet/C105871.pdf"
+		(property "Datasheet" "https://jlcpcb.com/api/file/downloadByFileSystemAccessId/8579705941367193600"
 			(at 139.7 194.31 0)
 			(effects
@@
 			)
 		)
-		(property "LCSC Part" "C105871"
+		(property "LCSC Part" "C25900"
+			(at 139.7 194.31 90)
+			(effects
+				(font
+					(size 1.27 1.27)
+				)
+				(hide yes)
+			)
+		)
+		(property "MPN" "0402WGF4701TCE"
 			(at 139.7 194.31 90)
 			(effects
@@
 			)
 		)
-		(property "MPN" "RC0402FR-074K7L"
+		(property "Manufacturer" "UNI-ROYAL(Uniroyal Elec)"
 			(at 139.7 194.31 90)
 			(effects
@@
 			)
 		)
-		(property "Datasheet" "https://www.lcsc.com/datasheet/C105871.pdf"
+		(property "Datasheet" "https://jlcpcb.com/api/file/downloadByFileSystemAccessId/8579705941367193600"
 			(at 209.55 194.31 0)
 			(effects
@@
 			)
 		)
-		(property "LCSC Part" "C105871"
+		(property "LCSC Part" "C25900"
+			(at 209.55 194.31 90)
+			(effects
+				(font
+					(size 1.27 1.27)
+				)
+				(hide yes)
+			)
+		)
+		(property "MPN" "0402WGF4701TCE"
 			(at 209.55 194.31 90)
 			(effects
@@
 			)
 		)
-		(property "MPN" "RC0402FR-074K7L"
+		(property "Manufacturer" "UNI-ROYAL(Uniroyal Elec)"
 			(at 209.55 194.31 90)
 			(effects
@@
 			)
 		)
-		(property "Datasheet" "https://www.lcsc.com/datasheet/C105875.pdf"
+		(property "Datasheet" "https://jlcpcb.com/api/file/downloadByFileSystemAccessId/8579706017514917888"
 			(at 265.43 179.07 0)
 			(effects
@@
 			)
 		)
-		(property "LCSC Part" "C105875"
+		(property "LCSC Part" "C25104"
 			(at 265.43 179.07 90)
 			(effects
@@
 			)
 		)
-		(property "MPN" "RC0402FR-07330RL"
+		(property "MPN" "0402WGF3300TCE"
+			(at 265.43 179.07 90)
+			(effects
+				(font
+					(size 1.27 1.27)
+				)
+				(hide yes)
+			)
+		)
+		(property "Manufacturer" "UNI-ROYAL(Uniroyal Elec)"
 			(at 265.43 179.07 90)
 			(effects
@@
 			)
 		)
-		(property "Datasheet" "https://www.lcsc.com/datasheet/C60490.pdf"
+		(property "Datasheet" "https://jlcpcb.com/api/file/downloadByFileSystemAccessId/8556212101498380288"
 			(at 41.91 185.42 0)
 			(effects
@@
 			)
 		)
-		(property "LCSC Part" "C60490"
+		(property "LCSC Part" "C25744"
+			(at 41.91 185.42 0)
+			(effects
+				(font
+					(size 1.27 1.27)
+				)
+				(hide yes)
+			)
+		)
+		(property "MPN" "0402WGF1002TCE"
 			(at 41.91 185.42 0)
 			(effects
@@
 			)
 		)
-		(property "MPN" "RC0402FR-0710KL"
+		(property "Manufacturer" "UNI-ROYAL(Uniroyal Elec)"
 			(at 41.91 185.42 0)
 			(effects
@@
 			)
 		)
-		(property "Datasheet" "https://www.lcsc.com/datasheet/C60474.pdf"
+		(property "Datasheet" "https://jlcpcb.com/api/file/downloadByFileSystemAccessId/8579707269996871680"
 			(at 53.34 132.08 0)
 			(effects
@@
 			)
 		)
-		(property "LCSC Part" "C60474"
+		(property "LCSC Part" "C1525"
+			(at 53.34 132.08 0)
+			(effects
+				(font
+					(size 1.27 1.27)
+				)
+				(hide yes)
+			)
+		)
+		(property "MPN" "CL05B104KO5NNNC"
 			(at 53.34 132.08 0)
 			(effects
@@
 			)
 		)
-		(property "MPN" "CC0402KRX7R7BB104"
+		(property "Manufacturer" "Samsung Electro-Mechanics"
 			(at 53.34 132.08 0)
 			(effects
