File: hardware/PicoDAC/PicoDAC.kicad_pcb (KiCad board)
At the start: 4 copper layers, 35.1 x 73.3 mm, 48 parts, among them CN1 PJ-327A 5JJ, U1 CS43131-CNZR, U2 XIAO-RP2350-DIP, U3 PCA9306DCUR, U4 SN74AXC4T245PWR, U5 XTPS7A2018, U7 74AHCT1G125GV

Commit message: added ground fill on top and bottom layer
Routing:
- net GND: track 132.4 -> 41.3 mm, vias 19 -> 88
- net /USB_GND: vias 2 -> 21
- added copper zone on B.Cu, net /USB_GND
- added copper zone on F.Cu, net /USB_GND
- added copper zone on B.Cu, net GND
- added copper zone on F.Cu, net GND
